File: charg.kicad_pcb (KiCad board)
At the start: 2 copper layers, 19 parts, among them IC1 SI3483DDV-T1-BE3, IC2 BQ25302RTER, J1 Vbus, J2 GND, J3 Vout, J4 EN, J5 Vbatt, J6 Therm, J7 GND, J8 STAT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

Commit message: Debloat
Parts:
- removed J3: Vout, TerminalBlock_MetzConnect:TerminalBlock_MetzConnect_360271_1x01_Horizontal_ScrewM3.0_Boxed
- removed J5: Vbatt, TerminalBlock_MetzConnect:TerminalBlock_MetzConnect_360271_1x01_Horizontal_ScrewM3.0_Boxed
- removed J6: Therm, TerminalBlock_MetzConnect:TerminalBlock_MetzConnect_360271_1x01_Horizontal_ScrewM3.0_Boxed
- removed J7: GND, TerminalBlock_MetzConnect:TerminalBlock_MetzConnect_360271_1x01_Horizontal_ScrewM3.0_Boxed
- removed J8: STAT, TerminalBlock_MetzConnect:TerminalBlock_MetzConnect_360271_1x01_Horizontal_ScrewM3.0_Boxed
- removed J9: REGN, TerminalBlock_MetzConnect:TerminalBlock_MetzConnect_360271_1x01_Horizontal_ScrewM3.0_Boxed
- J1: value Vbus -> Screw_Terminal_01x04; footprint TerminalBlock_MetzConnect:TerminalBlock_MetzConnect_360271_1x01_Horizontal_ScrewM3.0_Boxed -> Boost LTC3426:TerminalBlock_MetzConnect_Type059_RT06304HBWC_1x04_P3.50mm_Horizontal
- J2: value GND -> Screw_Terminal_01x04; footprint TerminalBlock_MetzConnect:TerminalBlock_MetzConnect_360271_1x01_Horizontal_ScrewM3.0_Boxed -> Boost LTC3426:TerminalBlock_MetzConnect_Type059_RT06304HBWC_1x04_P3.50mm_Horizontal
- moved R2 30.7 mm to (124.7, 76.8)
- moved C2 29.9 mm to (132.2, 76.2)
- moved C4 29.7 mm to (149.2, 65.5)
- moved C3 27.5 mm to (128.9, 76.7)
- moved J2 25.8 mm to (125.2, 62.0)
- moved J1 25.5 mm to (125.2, 70.6)
- moved C1 23.3 mm to (134.6, 76.2)
- moved D2 22.4 mm to (142.4, 68.7)
- moved C5 21.3 mm to (153.3, 59.6)
- moved J4 20.0 mm to (147.9, 69.0)
- moved IC2 18.9 mm to (148.7, 60.9)
- moved L1 18.9 mm to (141.4, 62.4)
- moved IC1 16.6 mm to (141.1, 73.2)
Connections:
- C2 pad 1: Net-(IC2-Pad2) -> Net-(C2-Pad1)
- C3 pad 1: Net-(IC2-Pad16) -> Net-(C3-Pad1)
- C5 pad 1: Net-(IC2-Pad10) -> Net-(C5-Pad1)
- IC1 pad 1: Net-(IC2-Pad10) -> Net-(C5-Pad1)
- IC1 pad 2: Net-(IC2-Pad10) -> Net-(C5-Pad1)
- IC1 pad 4: Net-(IC2-Pad16) -> Net-(C3-Pad1)
- IC1 pad 5: Net-(IC2-Pad10) -> Net-(C5-Pad1)
- IC1 pad 6: Net-(IC2-Pad10) -> Net-(C5-Pad1)
- IC2 pad 10: Net-(IC2-Pad10) -> Net-(C5-Pad1)
- IC2 pad 16: Net-(IC2-Pad16) -> Net-(C3-Pad1)
- IC2 pad 2: Net-(IC2-Pad2) -> Net-(C2-Pad1)
- J2 pad 1: Earth -> Net-(C3-Pad1)
- L1 pad 2: Net-(IC2-Pad10) -> Net-(C5-Pad1)

Commit message: Patch
Parts:
- C1, C2: footprint 2.2uF:CAPC0603X33N -> Library:CAPC0603X33N
- C3, C5: footprint 10uF MLCC:CAPC2012X94N -> Library:CAPC2012X94N
- C4: footprint 47nF:C1005_Commercial -> Library:C1005_Commercial
- D2: footprint Schottky dd:DIOM5026X220N -> Library:DIOM5026X220N
- IC1: footprint PFET:SOT95P284X110-6N -> Library:SOT95P284X110-6N
- IC2: footprint Charger bq 25302:QFN50P300X300X80-17N-D -> Library:QFN50P300X300X80-17N-D
- J1, J2: footprint Boost LTC3426:TerminalBlock_MetzConnect_Type059_RT06304HBWC_1x04_P3.50mm_Horizontal -> Library:TerminalBlock_MetzConnect_Type059_RT06304HBWC_1x04_P3.50mm_Horizontal
- J4: footprint Connector_PinHeader_1.00mm:PinHeader_1x01_P1.00mm_Vertical -> Library:PinHeader_1x01_P1.00mm_Vertical
- L1: footprint 1uH indc:IHHP0805ZHER1R0M01 -> Library:IHHP0805ZHER1R0M01
- R2: footprint 30k rst:RESC2012X70N -> Library:RESC2012X70N
- moved J2 53.7 mm to (178.4, 54.6), turned to -90 degrees
- moved C3 26.0 mm to (146.1, 57.1), turned to 90 degrees
- moved R2 24.1 mm to (144.8, 63.5), turned to 90 degrees
- moved IC1 24.0 mm to (152.4, 52.1), turned to 180 degrees
- moved C1 19.9 mm to (143.5, 58.4), turned to 90 degrees
- moved C2 19.2 mm to (143.5, 60.7), turned to 180 degrees
- moved D2 15.6 mm to (144.8, 53.3)
- moved J1 13.6 mm to (124.9, 57.0), turned to -90 degrees
- moved L1 11.0 mm to (151.1, 57.1)
- moved C4 8.43 mm to (148.3, 57.1), turned to 90 degrees
- moved J4 1.84 mm to (148.6, 67.3)
- moved C5 0.36 mm to (153.7, 59.7), turned to -90 degrees

Commit message: Update charg.kicad_pcb
Parts:
- moved J2 19.7 mm to (158.8, 54.6)
- moved J1 13.7 mm to (138.4, 54.6)
- moved IC1 1.27 mm to (152.4, 53.3)
- moved J4 1.27 mm to (148.6, 66.0)
Changed lines of the file:
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@@
   )
   (footprint "Library:SOT95P284X110-6N" (layer "F.Cu")
-    (at 152.4 52.07 180)
+    (at 152.4 53.34 180)
     (descr "SI3460DDV-T1-BE3")
     (tags "Integrated Circuit")
@@
   )
   (footprint "Library:TerminalBlock_MetzConnect_Type059_RT06304HBWC_1x04_P3.50mm_Horizontal" (layer "F.Cu")
-    (at 124.91 56.98 -90)
+    (at 138.43 54.61 -90)
     (descr "terminal block Metz Connect Type059_RT06304HBWC, 4 pins, pitch 3.5mm, size 14x6.5mm^2, drill diamater 1.2mm, pad diameter 2.3mm, see http://www.metz-connect.com/de/system/files/productfiles/Datenblatt_310591_RT063xxHBWC_OFF-022684T.pdf, script-generated using https://github.com/pointhi/kicad-footprint-generator/scripts/TerminalBlock_MetzConnect")
     (tags "THT terminal block Metz Connect Type059_RT06304HBWC pitch 3.5mm size 14x6.5mm^2 drill 1.2mm pad 2.3mm")
@@
   )
   (footprint "Library:TerminalBlock_MetzConnect_Type059_RT06304HBWC_1x04_P3.50mm_Horizontal" (layer "F.Cu")
-    (at 178.42 54.61 -90)
+    (at 158.75 54.61 -90)
     (descr "terminal block Metz Connect Type059_RT06304HBWC, 4 pins, pitch 3.5mm, size 14x6.5mm^2, drill diamater 1.2mm, pad diameter 2.3mm, see http://www.metz-connect.com/de/system/files/productfiles/Datenblatt_310591_RT063xxHBWC_OFF-022684T.pdf, script-generated using https://github.com/pointhi/kicad-footprint-generator/scripts/TerminalBlock_MetzConnect")
     (tags "THT terminal block Metz Connect Type059_RT06304HBWC pitch 3.5mm size 14x6.5mm^2 drill 1.2mm pad 2.3mm")
@@
   )
   (footprint "Library:PinHeader_1x01_P1.00mm_Vertical" (layer "F.Cu")
-    (at 148.59 67.31)
+    (at 148.59 66.04)
     (descr "Through hole straight pin header, 1x01, 1.00mm pitch, single row")
     (tags "Through hole pin header THT 1x01 1.00mm single row")

Commit message: No idea
Parts:
- C1, C2: footprint Library:CAPC0603X33N -> 2.2uF:CAPC0603X33N
- C3, C5: footprint Library:CAPC2012X94N -> 10uF MLCC:CAPC2012X94N
- C4: footprint Library:C1005_Commercial -> 47nF:C1005_Commercial
- D2: footprint Library:DIOM5026X220N -> Schottky dd:DIOM5026X220N
- IC1: footprint Library:SOT95P284X110-6N -> PFET:SOT95P284X110-6N
- IC2: footprint Library:QFN50P300X300X80-17N-D -> Charger bq 25302:QFN50P300X300X80-17N-D
- J1, J2: footprint Library:TerminalBlock_MetzConnect_Type059_RT06304HBWC_1x04_P3.50mm_Horizontal -> Boost LTC3426:TerminalBlock_MetzConnect_Type059_RT06304HBWC_1x04_P3.50mm_Horizontal
- J4: footprint Library:PinHeader_1x01_P1.00mm_Vertical -> Connector_PinHeader_1.00mm:PinHeader_1x01_P1.00mm_Vertical
- L1: footprint Library:IHHP0805ZHER1R0M01 -> 1uH indc:IHHP0805ZHER1R0M01
- R2: footprint Library:RESC2012X70N -> 30k rst:RESC2012X70N
- moved D2 2.64 mm to (145.5, 50.8), turned to 180 degrees
- moved C5 1.31 mm to (152.5, 60.3)
- moved IC1 1.27 mm to (152.4, 52.1), turned to 0 degrees
- moved L1 0.91 mm to (152.0, 57.1)
- moved C4 0.90 mm to (149.1, 56.6)
- moved C3 0.62 mm to (145.4, 57.1)
Connections:
- J1 pad 2: Earth -> Net-(C2-Pad1)
- J1 pad 3: Net-(C2-Pad1) -> Net-(IC2-Pad3)
- J1 pad 4: Net-(IC2-Pad3) -> Earth
Routing:
- net Net-(C3-Pad1): track 0.00 -> 17.4 mm
- net Net-(C5-Pad1): track 0.00 -> 7.05 mm
- net Net-(C1-Pad1): track 0.00 -> 6.66 mm
- net Net-(D2-Pad1): track 0.00 -> 4.62 mm

Commit message: PCB v1
Parts:
- moved D2 2.54 mm to (145.5, 53.3)
- moved J4 1.80 mm to (149.9, 64.8)
- moved R2 1.80 mm to (146.1, 64.8)
- moved C2 1.57 mm to (143.5, 62.2), turned to -90 degrees
- moved IC1 1.27 mm to (152.4, 53.3)
- moved C1 1.27 mm to (143.5, 59.7)
- moved C5 1.16 mm to (152.5, 61.4)
- moved C4 0.71 mm to (148.6, 57.1), turned to 0 degrees
- moved J2 0.45 mm to (159.2, 54.6)
- moved L1 0.36 mm to (152.4, 57.1)
- moved C3 0.16 mm to (145.6, 57.1), turned to 180 degrees
Routing:
- net Earth: track 0.00 -> 59.3 mm, vias 0 -> 5
- net Net-(C5-Pad1): track 7.05 -> 26.3 mm
- net Net-(IC2-Pad3): track 0.00 -> 13.0 mm
- net Net-(C1-Pad1): track 6.66 -> 18.8 mm
- net Net-(IC2-Pad7): track 0.00 -> 12.0 mm
- net Net-(C2-Pad1): track 0.00 -> 10.8 mm
- net Net-(IC2-Pad6): track 0.00 -> 2.98 mm
- net Net-(IC2-Pad4): track 0.00 -> 2.64 mm
- net Net-(C4-Pad1): track 0.00 -> 2.33 mm
- net Net-(D2-Pad1): track 4.62 -> 4.01 mm
- net Net-(C4-Pad2): track 0.00 -> 0.50 mm
- added copper zone on B.Cu, net Earth
- added copper zone on F.Cu, net Earth
- added copper zone on F.Cu, net Net-(C4-Pad2)
- added copper zone on F.Cu, net Net-(C5-Pad1)
Other:
- board outline added: 29.2 x 20.3 mm

Commit message: fill
filled earth
Routing:
- net Net-(C5-Pad1): track 26.3 -> 33.4 mm
- removed copper zone on B.Cu, net Earth
Changed lines of the file:
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@@
   (segment (start 148.4 57.36) (end 148.4 59.39) (width 0.25) (layer "F.Cu") (net 11))
   (segment (start 148.9 59.39) (end 149.4 59.39) (width 0.25) (layer "F.Cu") (net 12))
+  (segment (start 153.73 52.39) (end 151.13 52.39) (width 0.25) (layer "F.Cu") (net 13))
   (segment (start 153.28265 57.15) (end 153.28265 59.81625) (width 0.25) (layer "F.Cu") (net 13))
   (segment (start 151.9589 61.14) (end 152.4889 60.61) (width 0.25) (layer "F.Cu") (net 13))
@@
   (segment (start 150.15 61.14) (end 151.9589 61.14) (width 0.25) (layer "F.Cu") (net 13))
   (segment (start 153.28265 59.81625) (end 152.4889 60.61) (width 0.25) (layer "F.Cu") (net 13))
+  (segment (start 153.73 53.34) (end 151.13 53.34) (width 0.25) (layer "F.Cu") (net 13))
   (segment (start 153.73 52.39) (end 160.34 52.39) (width 0.25) (layer "F.Cu") (net 13))
   (segment (start 161.29 53.34) (end 161.29 56.02) (width 0.25) (layer "F.Cu") (net 13))
   (segment (start 153.28265 57.15) (end 158.24 57.15) (width 0.25) (layer "F.Cu") (net 13))
+  (segment (start 151.13 52.39) (end 151.13 53.34) (width 0.25) (layer "F.Cu") (net 13))
   (segment (start 158.24 57.15) (end 159.2 58.11) (width 0.25) (layer "F.Cu") (net 13))
+  (segment (start 153.73 52.39) (end 153.73 53.34) (width 0.25) (layer "F.Cu") (net 13))
   (segment (start 148.4 63.31) (end 148.4 62.39) (width 0.25) (layer "F.Cu") (net 14))
   (segment (start 149.86 64.77) (end 148.4 63.31) (width 0.25) (layer "F.Cu") (net 14))
@@
     )
   )
+  (zone (net 1) (net_name "Earth") (layer "F.Cu") (hatch edge 0.508)
+    (connect_pads (clearance 0.508))
+    (min_thickness 0.254) (filled_areas_thickness no)
+    (fill yes (thermal_gap 0.508) (thermal_bridge_width 0.508))
+    (polygon
+      (pts
+        (xy 162.56 69.85)
+        (xy 133.35 69.85)
+        (xy 133.35 49.53)
+        (xy 162.56 49.53)
+      )
+    )
+  )
   (zone (net 13) (net_name "Net-(C5-Pad1)") (layer "F.Cu") (hatch edge 0.508)
     (connect_pads (clearance 0.508))
@@
       )
     )
-  )
-  (zone (net 1) (net_name "Earth") (layer "B.Cu") (hatch edge 0.508)
-    (connect_pads (clearance 0.508))
-    (min_thickness 0.254) (filled_areas_thickness no)
-    (fill yes (thermal_gap 0.508) (thermal_bridge_width 0.508))
-    (polygon
-      (pts
-        (xy 144.78 64.77)
-        (xy 140.97 64.77)
-        (xy 140.97 54.61)
-        (xy 144.78 54.61)
-      )
-    )

Commit message: Patches + Fixes
Routing:
- net Earth: track 59.3 -> 34.0 mm
- net Net-(C5-Pad1): track 33.4 -> 19.4 mm
- net Net-(C1-Pad1): track 18.8 -> 19.5 mm
- added copper zone on B.Cu, net Earth
Other:
- board size 29.2 x 20.3 mm -> 29 x 20 mm
- board text added: "CubeSat EPS Battery Charger Module"
- board text added: "GEC Barton Hill"
