File: charg.kicad_pcb (KiCad board)
At the start: 2 copper layers, 29 x 20 mm, 13 parts, among them IC1 SI3483DDV-T1-BE3, IC2 BQ25302RTER, J1 Screw_Terminal_01x04, J2 Screw_Terminal_01x04, J4 EN

Commit message: DRC chk n' fix
Parts:
- moved C4 0.63 mm to (149.2, 57.1)
Routing:
- net Net-(C5-Pad1): track 19.4 -> 18.0 mm
Changed lines of the file:
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@@
   )
   (footprint "47nF:C1005_Commercial" (layer "F.Cu")
-    (at 148.59 57.15)
+    (at 149.225 57.15)
     (descr "C1005_Commercial")
     (tags "Capacitor")
@@
   (segment (start 158.88 54.29) (end 159.2 54.61) (width 0.25) (layer "F.Cu") (net 10))
   (segment (start 147.9 59.39) (end 147.9 58.65) (width 0.25) (layer "F.Cu") (net 10))
-  (segment (start 148.19 57.15) (end 148.4 57.36) (width 0.25) (layer "F.Cu") (net 11))
-  (segment (start 148.4 57.36) (end 148.4 59.39) (width 0.25) (layer "F.Cu") (net 11))
+  (segment (start 148.4 59.39) (end 148.4 57.575) (width 0.25) (layer "F.Cu") (net 11))
+  (segment (start 148.4 57.575) (end 148.825 57.15) (width 0.25) (layer "F.Cu") (net 11))
   (segment (start 148.9 59.39) (end 149.4 59.39) (width 0.25) (layer "F.Cu") (net 12))
   (segment (start 159.2 58.11) (end 161.59 55.72) (width 0.52) (layer "F.Cu") (net 13))
@@
   (segment (start 151.9589 61.14) (end 152.4889 60.61) (width 0.29) (layer "F.Cu") (net 13))
   (segment (start 161.59 52.65) (end 160.09 51.15) (width 0.52) (layer "F.Cu") (net 13))
-  (segment (start 158.24 57.15) (end 159.2 58.11) (width 0.29) (layer "F.Cu") (net 13))
   (segment (start 150.15 61.14) (end 151.9589 61.14) (width 0.29) (layer "F.Cu") (net 13))
   (segment (start 154.85 52.39) (end 153.73 52.39) (width 0.52) (layer "F.Cu") (net 13))

Commit message: FInal...I guess
Parts:
- D2: footprint Schottky dd:DIOM5026X220N -> Schottky DD with stock:DIOM5126X265N
- moved J2 10.4 mm to (158.3, 64.9), turned to 90 degrees
Connections:
- J2 pad 1: Net-(C3-Pad1) -> Earth
- J2 pad 2: Net-(C5-Pad1) -> Net-(IC2-Pad7)
- J2 pad 3: Net-(IC2-Pad7) -> Net-(C5-Pad1)
- J2 pad 4: Earth -> Net-(C3-Pad1)
Routing:
- net Earth: track 34.0 -> 36.2 mm
- net Net-(C5-Pad1): track 18.0 -> 16.5 mm
- net Net-(C3-Pad1): track 17.5 -> 16.5 mm
- net Net-(IC2-Pad7): track 12.0 -> 11.1 mm

Commit message: Replace 30k ISEt with 30.9k
Parts:
- R2: value 30k -> 30.9k; footprint 30k rst:RESC2012X70N -> rst 30.9k:RC0603FR-0730K9L
Changed lines of the file:
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@@
   (net 13 "Net-(C5-Pad1)")
   (net 14 "Net-(IC2-Pad6)")
-  (footprint "30k rst:RESC2012X70N" (layer "F.Cu")
+  (footprint "rst 30.9k:RC0603FR-0730K9L" (layer "F.Cu")
     (at 146.05 64.77 90)
-    (descr "ERJ-PB6B3002V")
-    (tags "Resistor")
     (property "Sheetfile" "charg.kicad_sch")
     (property "Sheetname" "")
-    (attr smd)
-    (fp_text reference "R2" (at 0.12 1.54 90) (layer "F.SilkS")
-      (effects (font (size 0.6 0.6) (thickness 0.15)))
+    (attr through_hole)
+    (fp_text reference "R2" (at 0 0 90) (layer "F.SilkS") hide
+      (effects (font (size 1 1) (thickness 0.15)))
     )
-    (fp_text value "30k" (at 0 0 90) (layer "F.SilkS") hide
-      (effects (font (size 1.27 1.27) (thickness 0.254)))
+    (fp_text value "30.9k" (at 0 0 90) (layer "F.SilkS") hide
+      (effects (font (size 1 1) (thickness 0.15)))
     )
-    (fp_text user "${REFERENCE}" (at 0 0 90) (layer "F.Fab")
-      (effects (font (size 1.27 1.27) (thickness 0.254)))
+    (fp_text user "*" (at 0 0 90) (layer "F.SilkS") hide
+      (effects (font (size 1 1) (thickness 0.15)))
     )
-    (fp_line (start 0 -0.525) (end 0 0.525) (layer "F.SilkS") (width 0.2))
-    (fp_line (start 1.725 0.95) (end -1.725 0.95) (layer "F.CrtYd") (width 0.05))
-    (fp_line (start -1.725 -0.95) (end 1.725 -0.95) (layer "F.CrtYd") (width 0.05))
-    (fp_line (start 1.725 -0.95) (end 1.725 0.95) (layer "F.CrtYd") (width 0.05))
-    (fp_line (start -1.725 0.95) (end -1.725 -0.95) (layer "F.CrtYd") (width 0.05))
-    (fp_line (start -1 0.625) (end -1 -0.625) (layer "F.Fab") (width 0.1))
-    (fp_line (start 1 -0.625) (end 1 0.625) (layer "F.Fab") (width 0.1))
-    (fp_line (start -1 -0.625) (end 1 -0.625) (layer "F.Fab") (width 0.1))
-    (fp_line (start 1 0.625) (end -1 0.625) (layer "F.Fab") (width 0.1))
-    (pad "1" smd rect (at -0.95 0 90) (size 1.05 1.4) (layers "F.Cu" "F.Paste" "F.Mask")
+    (fp_text user "Copyright 2021 Accelerated Designs. All rights reserved." (at 0 0 90) (layer "Cmts.User")
+      (effects (font (size 0.127 0.127) (thickness 0.002)))
+    )
+    (fp_text user "0.091in/2.311mm" (at 0 -3.4544 90) (layer "Cmts.User") hide
+      (effects (font (size 1 1) (thickness 0.15)))
+    )
+    (fp_text user "0.032in/0.813mm" (at 3.8481 0 90) (layer "Cmts.User")
+      (effects (font (size 1 1) (thickness 0.15)))
+    )
+    (fp_text user "0.031in/0.787mm" (at 0 3.4544 90) (layer "Cmts.User") hide
+      (effects (font (size 1 1) (thickness 0.15)))
+    )
+    (fp_text user "*" (at 0 0 90) (layer "F.Fab")
+      (effects (font (size 1 1) (thickness 0.15)))
+    )
+    (fp_line (start 0.08615 -0.5334) (end -0.08615 -0.5334) (layer "F.SilkS") (width 0.12))
+    (fp_line (start -0.08615 0.5334) (end 0.08615 0.5334) (layer "F.SilkS") (width 0.12))
+    (fp_line (start -1.0541 -3.0734) (end -1.0541 -2.8194) (layer "Cmts.User") (width 0.1))
+    (fp_line (start -0.8001 -2.9464) (end -1.0541 -2.8194) (layer "Cmts.User") (width 0.1))
+    (fp_line (start 3.3401 -0.4064) (end 3.4671 -0.6604) (layer "Cmts.User") (width 0.1))
+    (fp_line (start 0.3937 2.9464) (end -0.8763 2.9464) (layer "Cmts.User") (width 0.1))
+    (fp_line (start 1.0541 2.8194) (end 1.0541 3.0734) (layer "Cmts.User") (width 0.1))
+    (fp_line (start 0.8001 2.9464) (end 1.0541 2.8194) (layer "Cmts.User") (width 0.1))
+    (fp_line (start -0.8001 0) (end -0.8001 -3.3274) (layer "Cmts.User") (width 0.1))
+    (fp_line (start 3.3401 -0.4064) (end 3.3401 -1.6764) (layer "Cmts.User") (width 0.1))
+    (fp_line (start 0.8001 2.9464) (end 2.0701 2.9464) (layer "Cmts.User") (width 0.1))
+    (fp_line (start 0 0.4064) (end 3.7211 0.4064) (layer "Cmts.User") (width 0.1))
+    (fp_line (start 0.3937 0) (end 0.3937 3.3274) (layer "Cmts.User") (width 0.1))
+    (fp_line (start 3.3401 0.4064) (end 3.3401 1.6764) (layer "Cmts.User") (width 0.1))
+    (fp_line (start 0.8001 -2.9464) (end 1.0541 -2.8194) (layer "Cmts.User") (width 0.1))
+    (fp_line (start 0.1397 2.8194) (end 0.1397 3.0734) (layer "Cmts.User") (width 0.1))
+    (fp_line (start 1.0541 -3.0734) (end 1.0541 -2.8194) (layer "Cmts.User") (width 0.1))
+    (fp_line (start -0.8001 -2.9464) (end -1.0541 -3.0734) (layer "Cmts.User") (width 0.1))
+    (fp_line (start 0.8001 0) (end 0.8001 -3.3274) (layer "Cmts.User") (width 0.1))
+    (fp_line (start 0.3937 2.9464) (end 0.1397 2.8194) (layer "Cmts.User") (width 0.1))
+    (fp_line (start 3.3401 0.4064) (end 3.4671 0.6604) (layer "Cmts.User") (width 0.1))
+    (fp_line (start -0.8001 -2.9464) (end -2.0701 -2.9464) (layer "Cmts.User") (width 0.1))
+    (fp_line (start 0.8001 -2.9464) (end 1.0541 -3.0734) (layer "Cmts.User") (width 0.1))
+    (fp_line (start 0.8001 0) (end 0.8001 3.3274) (layer "Cmts.User") (width 0.1))
+    (fp_line (start 0 -0.4064) (end 3.7211 -0.4064) (layer "Cmts.User") (width 0.1))
+    (fp_line (start 0.8001 -2.9464) (end 2.0701 -2.9464) (layer "Cmts.User") (width 0.1))
+    (fp_line (start 0.3937 2.9464) (end 0.1397 3.0734) (layer "Cmts.User") (width 0.1))
+    (fp_line (start 3.3401 -0.4064) (end 3.2131 -0.6604) (layer "Cmts.User") (width 0.1))
+    (fp_line (start 0.8001 2.9464) (end 1.0541 3.0734) (layer "Cmts.User") (width 0.1))
+    (fp_line (start 3.2131 0.6604) (end 3.4671 0.6604) (layer "Cmts.User") (width 0.1))
+    (fp_line (start 3.3401 0.4064) (end 3.2131 0.6604) (layer "Cmts.User") (width 0.1))
+    (fp_line (start 3.2131 -0.6604) (end 3.4671 -0.6604) (layer "Cmts.User") (width 0.1))
+    (fp_line (start -1.4097 -0.6604) (end 1.4097 -0.6604) (layer "F.CrtYd") (width 0.05))
+    (fp_line (start -1.4097 0.6604) (end -1.4097 -0.6604) (layer "F.CrtYd") (width 0.05))
+    (fp_line (start 1.4097 -0.6604) (end 1.4097 0.6604) (layer "F.CrtYd") (width 0.05))
+    (fp_line (start -1.4097 -0.6604) (end 1.4097 -0.6604) (layer "F.CrtYd") (width 0.05))
+    (fp_line (start 1.4097 0.6604) (end -1.4097 0.6604) (layer "F.CrtYd") (width 0.05))
+    (fp_line (start 1.4097 -0.6604) (end 1.4097 0.6604) (layer "F.CrtYd") (width 0.05))
+    (fp_line (start 1.4097 0.6604) (end -1.4097 0.6604) (layer "F.CrtYd") (width 0.05))
+    (fp_line (start -1.4097 0.6604) (end -1.4097 -0.6604) (layer "F.CrtYd") (width 0.05))
+    (fp_line (start -0.3937 0.4064) (end -0.3937 -0.4064) (layer "F.Fab") (width 0.1))
+    (fp_line (start -0.8001 -0.4064) (end -0.8001 0.4064) (layer "F.Fab") (width 0.1))
+    (fp_line (start 0.8001 0.4064) (end 0.8001 -0.4064) (layer "F.Fab") (width 0.1))
+    (fp_line (start 0.8001 -0.4064) (end 0.3937 -0.4064) (layer "F.Fab") (width 0.1))
+    (fp_line (start 0.3937 -0.4064) (end 0.3937 0.4064) (layer "F.Fab") (width 0.1))
+    (fp_line (start 0.8001 0.4064) (end 0.8001 -0.4064) (layer "F.Fab") (width 0.1))
+    (fp_line (start -0.8001 0.4064) (end 0.8001 0.4064) (layer "F.Fab") (width 0.1))
+    (fp_line (start 0.8001 -0.4064) (end -0.8001 -0.4064) (layer "F.Fab") (width 0.1))
+    (fp_line (start 0.3937 0.4064) (end 0.8001 0.4064) (layer "F.Fab") (width 0.1))
+    (fp_line (start -0.8001 -0.4064) (end -0.8001 0.4064) (layer "F.Fab") (width 0.1))
+    (fp_line (start -0.3937 -0.4064) (end -0.8001 -0.4064) (layer "F.Fab") (width 0.1))
+    (fp_line (start -0.8001 0.4064) (end -0.3937 0.4064) (layer "F.Fab") (width 0.1))
+    (pad "1" smd rect (at -0.7747 0 90) (size 0.762 0.8128) (layers "F.Cu" "F.Paste" "F.Mask")
       (net 1 "Earth") (pintype "passive"))
-    (pad "2" smd rect (at 0.95 0 90) (size 1.05 1.4) (layers "F.Cu" "F.Paste" "F.Mask")
+    (pad "2" smd rect (at 0.7747 0 90) (size 0.762 0.8128) (layers "F.Cu" "F.Paste" "F.Mask")
       (net 4 "Net-(IC2-Pad4)") (pintype "passive"))
-    (model "ERJ-PB6B3002V.stp" hide
+    (model "/mnt/DAA829C1A8299CCF/EEE/S7/PROJ/COMPS/RST/30.9k/ul_RC0603FR-0730K9L/KiCAD/2022-12-29_14-17-30/2022-12-29_14-17-30.lib" hide
       (offset (xyz 0 0 0))
       (scale (xyz 1 1 1))
       (rotate (xyz 0 0 0))
     )
-    (model "/mnt/DAA829C1A8299CCF/EEE/S7/PROJ/COMPS/RST/30k/LIB_ERJ-PB6B3002V/ERJ-PB6B3002V/3D/ERJ-PB6B3002V.stp"
+    (model "/mnt/DAA829C1A8299CCF/EEE/S7/PROJ/COMPS/RST/30.9k/ul_RC0603FR-0730K9L/2022-12-29_14-17-29/STEP/RC0603N_YAG.step"
       (offset (xyz 0 0 0))
       (scale (xyz 1 1 1))

Commit message: Update Gerbuhs
Parts:
- moved L1 0.90 mm to (151.8, 57.8)
- moved C4 0.90 mm to (148.6, 56.5)
Routing:
- net Net-(C4-Pad1): track 2.42 -> 3.16 mm
- net Earth: vias 5 -> 8
Other:
- board text added: "Battery Charger Module"
- board text added: "GECB"
- board text removed: "CubeSat EPS Battery Charger Module"
- board text removed: "GEC Barton Hill"
Changed lines of the file:
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@@
   )
   (footprint "47nF:C1005_Commercial" (layer "F.Cu")
-    (at 149.225 57.15)
+    (at 148.59 56.515)
     (descr "C1005_Commercial")
     (tags "Capacitor")
@@
   )
   (footprint "1uH indc:IHHP0805ZHER1R0M01" (layer "F.Cu")
-    (at 152.4 57.15)
+    (at 151.765 57.785)
     (property "Sheetfile" "charg.kicad_sch")
     (property "Sheetname" "")
@@
   (gr_arc (start 158.59 50.15) (mid 161.418427 51.321573) (end 162.59 54.15) (layer "Edge.Cuts") (width 0.1))
   (gr_line (start 158.59 70.15) (end 137.59 70.15) (layer "Edge.Cuts") (width 0.1))
-  (gr_text "GEC Barton Hill" (at 154.178 68.834) (layer "F.SilkS")
+  (gr_text "GECB" (at 148.59 69.215) (layer "F.SilkS")
     (effects (font (size 0.7 0.7) (thickness 0.15)))
   )
-  (gr_text "CubeSat EPS Battery Charger Module" (at 145.542 67.818) (layer "F.SilkS")
+  (gr_text "Battery Charger Module" (at 148.59 67.818) (layer "F.SilkS")
     (effects (font (size 0.7 0.7) (thickness 0.1)))
   )
+  (segment (start 148.966 60.574) (end 149.22 60.32) (width 0.25) (layer "F.Cu") (net 1))
   (segment (start 147.635 65.72) (end 148.59 66.675) (width 0.25) (layer "F.Cu") (net 1))
   (segment (start 146.05 65.72) (end 147.635 65.72) (width 0.25) (layer "F.Cu") (net 1))
@@
   (segment (start 150.74 62.23) (end 150.15 61.64) (width 0.25) (layer "F.Cu") (net 1))
   (segment (start 153.5 64.94) (end 153.035 65.405) (width 0.25) (layer "F.Cu") (net 1))
-  (segment (start 149.4 61.64) (end 148.65 60.89) (width 0.25) (layer "F.Cu") (net 1))
+  (segment (start 149.4 61.64) (end 149.036 61.276) (width 0.25) (layer "F.Cu") (net 1))
   (segment (start 148.59 66.675) (end 156.565 66.675) (width 0.25) (layer "F.Cu") (net 1))
   (segment (start 158.3 64.94) (end 153.5 64.94) (width 0.25) (layer "F.Cu") (net 1))
   (segment (start 143.51 62.56) (end 143.51 63.5) (width 0.35) (layer "F.Cu") (net 1))
-  (segment (start 148.65 60.89) (end 149.4 60.14) (width 0.25) (layer "F.Cu") (net 1))
+  (segment (start 148.65 60.89) (end 148.966 60.574) (width 0.25) (layer "F.Cu") (net 1))
+  (segment (start 149.036 61.276) (end 148.65 60.89) (width 0.25) (layer "F.Cu") (net 1))
   (segment (start 156.565 66.675) (end 158.3 64.94) (width 0.25) (layer "F.Cu") (net 1))
   (segment (start 152.4889 62.23) (end 150.74 62.23) (width 0.25) (layer "F.Cu") (net 1))
   (segment (start 146.05 65.72) (end 139.04 65.72) (width 0.25) (layer "F.Cu") (net 1))
+  (segment (start 149.22 60.32) (end 149.4 60.14) (width 0.25) (layer "F.Cu") (net 1))
   (segment (start 139.04 65.72) (end 138.43 65.11) (width 0.25) (layer "F.Cu") (net 1))
   (segment (start 150.15 61.64) (end 149.4 61.64) (width 0.25) (layer "F.Cu") (net 1))
-  (via (at 148.65 60.89) (size 0.8) (drill 0.4) (layers "F.Cu" "B.Cu") (net 1))
+  (via (at 149.036 61.276) (size 0.6) (drill 0.4) (layers "F.Cu" "B.Cu") (net 1))
   (via (at 143.51 57.15) (size 0.8) (drill 0.4) (layers "F.Cu" "B.Cu") (free) (net 1))
+  (via (at 148.082 61.214) (size 0.6) (drill 0.4) (layers "F.Cu" "B.Cu") (net 1))
   (via (at 154.305 62.23) (size 0.8) (drill 0.4) (layers "F.Cu" "B.Cu") (free) (net 1))
   (via (at 143.51 63.5) (size 0.8) (drill 0.4) (layers "F.Cu" "B.Cu") (free) (net 1))
   (via (at 153.035 65.405) (size 0.8) (drill 0.4) (layers "F.Cu" "B.Cu") (free) (net 1))
+  (via (at 148.082 60.452) (size 0.6) (drill 0.4) (layers "F.Cu" "B.Cu") (net 1))
+  (via (at 148.966 60.574) (size 0.6) (drill 0.4) (layers "F.Cu" "B.Cu") (net 1))
   (segment (start 148.46 54.29) (end 147.51 53.34) (width 0.52) (layer "F.Cu") (net 2))
   (segment (start 151.13 54.29) (end 148.46 54.29) (width 0.52) (layer "F.Cu") (net 2))
@@
   (segment (start 158.15 54.29) (end 158.3 54.44) (width 0.25) (layer "F.Cu") (net 10))
   (segment (start 147.9 59.39) (end 147.9 58.65) (width 0.25) (layer "F.Cu") (net 10))
-  (segment (start 148.4 59.39) (end 148.4 57.575) (width 0.25) (layer "F.Cu") (net 11))
-  (segment (start 148.4 57.575) (end 148.825 57.15) (width 0.25) (layer "F.Cu") (net 11))
+  (segment (start 147.955 57.785) (end 147.955 56.75) (width 0.25) (layer "F.Cu") (net 11))
+  (segment (start 148.4 58.23) (end 147.955 57.785) (width 0.25) (layer "F.Cu") (net 11))
+  (segment (start 147.955 56.75) (end 148.19 56.515) (width 0.25) (layer "F.Cu") (net 11))
+  (segment (start 148.4 59.39) (end 148.4 58.23) (width 0.25) (layer "F.Cu") (net 11))
   (segment (start 148.9 59.39) (end 149.4 59.39) (width 0.25) (layer "F.Cu") (net 12))
   (segment (start 156.09 51.15) (end 158.465 51.15) (width 0.52) (layer "F.Cu") (net 13))
@@
     (polygon
       (pts
-        (xy 151.9 57.15)
+        (xy 151.13 57.15)
         (xy 151.13 58.42)
-        (xy 151.13 59.69)
-        (xy 148.59 59.69)
+        (xy 149.86 59.69)
+        (xy 148.702056 59.69)
         (xy 148.59 55.88)
-        (xy 151.9 55.88)
+        (xy 150.495 55.88)
       )
     )
@@
     (polygon
       (pts
-        (xy 159.09 59.65)
-        (xy 157.09 59.65)
-        (xy 157.09 61.15)
+        (xy 159.09 59.055)
+        (xy 157.09 59.69)
+        (xy 155.575 61.15)
         (xy 151.59 61.15)
         (xy 151.59 59.15)
-        (xy 152.59 59.15)
-        (xy 152.59 56.277)
+        (xy 151.955 59.15)
+        (xy 151.955 56.277)
         (xy 159.09 56.277)
       )
