File: charg.kicad_sch (KiCad schematic)
At the start: 13 parts, among them IC1 SI3483DDV-T1-BE3, IC2 BQ25302RTER, J1 Screw_Terminal_01x04, J2 Screw_Terminal_01x04, J4 EN

Commit message: Update charg.kicad_sch
Parts:
- D2: value RBR3L40ADD -> STPS2150A
Changed lines of the file:
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@@
     (in_bom yes) (on_board yes)
     (property "Reference" "D2" (id 0) (at 156.21 68.58 0))
-    (property "Value" "RBR3L40ADD" (id 1) (at 157.48 73.66 0))
+    (property "Value" "STPS2150A" (id 1) (at 157.48 73.66 0))
     (property "Footprint" "Schottky DD with stock:DIOM5126X265N" (id 2) (at 156.21 71.12 0)
       (effects (font (size 1.27 1.27)) hide)
@@
     )
     (path "/64e04f30-b75a-485a-9e25-e618219d18d5"
-      (reference "D2") (unit 1) (value "RBR3L40ADD") (footprint "Schottky DD with stock:DIOM5126X265N")
+      (reference "D2") (unit 1) (value "STPS2150A") (footprint "Schottky DD with stock:DIOM5126X265N")
     )
     (path "/ff90fce7-88c8-4858-850a-5a7e1e5af2e0"

Commit message: Add thermy rsts
Parts:
- added R1: 4.52k, rst 30.9k:RC0603FR-0730K9L, symbol Device:R_US
- added R3: 23.6k, rst 30.9k:RC0603FR-0730K9L, symbol Device:R_US
Connections:
- net Earth: now also R3.1
- net REGN: now reaches C2.1, IC2.2 (REGN), J1.2 (Pin_2)
- net REGN: now also R1.2
- net at IC2.7 (TS), J2.2 (Pin_2): now also R1.1, R3.2
Other:
- moved on the sheet: J2
